Commit message: add parallel_joint

File: wpb_arm_description/urdf/wpb_arm_1.urdf (robot description, URDF)
Before this commit: robot wpb_arm_1, 6 links, 5 joints
Links:
- added link upper_parallel_link
Joints:
- added joint upper_parallel_joint: type revolute, parent upper_arm_link, child upper_parallel_link, origin xyz=0 0 0.115, axis 0 1 0, limit lower=-1.57 upper=1.57 effort=1000.0 velocity=0.5, mimic joint=joint_1 multiplier=-1 offset=0
- joint joint_2: axis 0 1 0 -> 0 -1 0; origin xyz=0 0 0.115 rpy=0 0 0 -> xyz=0 0 0 rpy=0 0 0; parent upper_arm_link -> upper_parallel_link
- joint joint_4: axis 0 1 0 -> 0 -1 0
